File: KiCad/GR_RS485_DMX_Breakout.kicad_pcb (KiCad board)
At the start: 2 copper layers, 46.8 x 26.4 mm, 20 parts, among them J1 Conn_01x06, J2 XLR3, J3 Conn_01x02, U1 CRE1S0505SC, U2 ADM2483xRW, U3 ADM809

Commit message: Add files via upload
Changed lines of the file:
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@@
   )
   (setup
-    (last_trace_width 0.254)
+    (last_trace_width 0.25)
     (user_trace_width 0.2032)
     (user_trace_width 0.254)
@@
     (mod_text_size 0.8 0.8)
     (mod_text_width 0.15)
-    (pad_size 3.2 3.2)
-    (pad_drill 3.2)
+    (pad_size 1.5 2)
+    (pad_drill 0.9)
     (pad_to_mask_clearance 0)
     (aux_axis_origin 180.211 146.771)
@@
     (fp_line (start -0.25 -2.27) (end -1.45 -2.27) (layer F.SilkS) (width 0.12))
     (fp_line (start -1.45 -2.27) (end -1.45 -1.07) (layer F.SilkS) (width 0.12))
-    (pad 4 thru_hole oval (at 0 7.62) (size 1.5 2) (drill 0.7) (layers *.Cu *.Mask)
+    (pad 4 thru_hole oval (at 0 7.62) (size 1.5 2) (drill 0.9) (layers *.Cu *.Mask)
       (net 5 VCC))
-    (pad 3 thru_hole oval (at 0 5.08) (size 1.5 2) (drill 0.7) (layers *.Cu *.Mask)
+    (pad 3 thru_hole oval (at 0 5.08) (size 1.5 2) (drill 0.9) (layers *.Cu *.Mask)
       (net 4 GND))
-    (pad 2 thru_hole oval (at 0 2.54) (size 1.5 2) (drill 0.7) (layers *.Cu *.Mask)
+    (pad 2 thru_hole oval (at 0 2.54) (size 1.5 2) (drill 0.9) (layers *.Cu *.Mask)
       (net 2 +5V))
-    (pad 1 thru_hole rect (at 0 0) (size 1.5 2) (drill 0.7) (layers *.Cu *.Mask)
+    (pad 1 thru_hole rect (at 0 0) (size 1.5 2) (drill 0.9) (layers *.Cu *.Mask)
       (net 1 GNDREF))
     (model ${KISYS3DMOD}/Converter_DCDC.3dshapes/Converter_DCDC_muRata_CRE1xxxxxxSC_THT.wrl
@@
   (segment (start 204.646 143.606) (end 204.646 142.121) (width 0.254) (layer F.Cu) (net 11))
   (segment (start 205.061 144.021) (end 204.646 143.606) (width 0.254) (layer F.Cu) (net 11))
-  (segment (start 203.921 139.206) (end 204.211 139.496) (width 0.254) (layer F.Cu) (net 17))
   (segment (start 214.171 137.571) (end 214.171 134.131) (width 0.254) (layer F.Cu) (net 12))
   (segment (start 214.171 134.131) (end 209.811 129.771) (width 0.254) (layer F.Cu) (net 12))
@@
   (segment (start 206.9735 136.4085) (end 205.911 137.471) (width 0.254) (layer F.Cu) (net 13))
   (segment (start 208.411 134.971) (end 206.9735 136.4085) (width 0.254) (layer F.Cu) (net 13))
+  (segment (start 203.921 139.206) (end 204.211 139.496) (width 0.254) (layer F.Cu) (net 17))
   (segment (start 204.211 139.496) (end 206.361 139.496) (width 0.254) (layer F.Cu) (net 17))
   (segment (start 207.186 140.321) (end 207.186 142.121) (width 0.254) (layer F.Cu) (net 17))
