File: KiCad/GR_RS485_DMX_Breakout.sch (KiCad schematic (older format))
At the start: 19 parts, among them J1 Conn_01x06, J2 XLR3, J3 Conn_01x02, U1 CRE1S0505SC, U2 ADM2483xRW, U3 ADM809

Commit message: Add files via upload
Parts:
- R3, R4: value DNI -> 0r
- R5, R6: value 0r -> DNI
Other:
- note added: "Default Config: Receiver"
- note removed: "Default Config: Transmitter"
Changed lines of the file:
@@
 Sheet 1 1
 Title "DMX Interface"
-Date "2023-11-13"
+Date "2023-11-23"
 Rev "1"
 Comp "Gadget Reboot"
@@
 P 8100 4050
 F 0 "R4" V 8050 3950 50  0000 R CNN
-F 1 "DNI" V 8050 4200 50  0000 R CNN
+F 1 "0r" V 8050 4200 50  0000 R CNN
 F 2 "Resistor_SMD:R_0805_2012Metric_Pad1.15x1.40mm_HandSolder" H 8100 4050 50  0001 C CNN
 F 3 "~" H 8100 4050 50  0001 C CNN
@@
 P 8100 4200
 F 0 "R6" V 8050 4100 50  0000 R CNN
-F 1 "0r" V 8050 4350 50  0000 R CNN
+F 1 "DNI" V 8050 4350 50  0000 R CNN
 F 2 "Resistor_SMD:R_0805_2012Metric_Pad1.15x1.40mm_HandSolder" H 8100 4200 50  0001 C CNN
 F 3 "~" H 8100 4200 50  0001 C CNN
@@
 P 7025 4200
 F 0 "R5" V 6975 4100 50  0000 R CNN
-F 1 "0r" V 6975 4350 50  0000 R CNN
+F 1 "DNI" V 6975 4350 50  0000 R CNN
 F 2 "Resistor_SMD:R_0805_2012Metric_Pad1.15x1.40mm_HandSolder" H 7025 4200 50  0001 C CNN
 F 3 "~" H 7025 4200 50  0001 C CNN
@@
 P 7025 4050
 F 0 "R3" V 6975 3950 50  0000 R CNN
-F 1 "DNI" V 6975 4200 50  0000 R CNN
+F 1 "0r" V 6975 4200 50  0000 R CNN
 F 2 "Resistor_SMD:R_0805_2012Metric_Pad1.15x1.40mm_HandSolder" H 7025 4050 50  0001 C CNN
 F 3 "~" H 7025 4050 50  0001 C CNN
@@
 Termination \nJumper
 Text Notes 6825 3725 0    70   ~ 0
-Default Config: Transmitter
+Default Config: Receiver
 $EndSCHEMATC
